File: hardware/stm8-accelerometer -1.brd (EAGLE design)
At the start: 15 parts, among them U1 MCP1700T-3302E, U2 STM8SX03F3, U3 MPU6050

Commit message: Clean up.  Still WIP
Parts:
- added R4: 0R, ipc-7351-resistor:RESC3115X70N
- moved LICENSE1 5.83 mm to (5.13, 11.3)
Connections:
- new net N$1: R4.2, U3.2
- net GND: now also R4.1; no longer U3.2
Routing:
- net N$1: track 0.00 -> 7.99 mm
- net GND: track 14.0 -> 9.67 mm
- added copper zone on layer 1, net N$1
Other:
- board text removed: "Jumper"
Changed lines of the file:
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@@
 <wire x1="21.463" y1="0" x2="0" y2="0" width="0.127" layer="51"/>
 <wire x1="0" y1="0" x2="0" y2="37.0332" width="0.127" layer="51"/>
-<wire x1="4.953" y1="10.9728" x2="6.9596" y2="13.0048" width="0.4064" layer="51"/>
 <text x="0.4064" y="16.4846" size="0.6096" layer="21" ratio="15">Copyright (c)
 2021 by
@@
 <text x="15.1892" y="16.6878" size="0.8128" layer="21" ratio="15">STM8
 Gyrostick</text>
-<text x="4.6228" y="11.2776" size="0.6096" layer="51" rot="R45">Jumper</text>
 <wire x1="10.7442" y1="10.9728" x2="10.7442" y2="24.9428" width="0" layer="51"/>
 <text x="5.08" y="-3.81" size="0.6096" layer="51">MPU6050 dimensions are
@@
 <element name="H1" library="holes" package="3,0-PAD" value="MOUNT-PAD-ROUND3.0" x="10.7442" y="16.256" smashed="yes"/>
 <element name="U3" library="misc pcb" package="MPU6050" value="MPU6050" x="10.7442" y="22.5044" rot="R90"/>
-<element name="LICENSE1" library="Misc logo" package="CC-BY-50" value="CC-BY50%" x="0.381" y="14.6558"/>
+<element name="LICENSE1" library="Misc logo" package="CC-BY-50" value="CC-BY50%" x="5.1308" y="11.2776"/>
+<element name="R4" library="ipc-7351-resistor" package="RESC3115X70N" value="0R" x="2.54" y="14.6812" smashed="yes">
+<attribute name="NAME" x="5.0104" y="14.3763" size="0.6096" layer="25" font="vector" ratio="15"/>
+<attribute name="VALUE" x="0.54" y="12.2937" size="1.27" layer="27" font="vector" ratio="10"/>
+</element>
 </elements>
 <signals>
@@
 <wire x1="17.607" y1="9.23" x2="16.215" y2="9.23" width="0.3048" layer="1"/>
 <wire x1="16.215" y1="9.23" x2="16.002" y2="9.017" width="0.3048" layer="1"/>
-<contactref element="U3" pad="2"/>
-<wire x1="4.3942" y1="22.5044" x2="4.3942" y2="18.7452" width="0.4064" layer="1"/>
-<wire x1="4.3942" y1="18.7452" x2="4.064" y2="18.415" width="0.4064" layer="1"/>
-<wire x1="6.9596" y1="13.0302" x2="6.9342" y2="13.0048" width="0.4064" layer="1"/>
-<wire x1="4.9784" y1="10.9982" x2="4.953" y2="10.9728" width="0.4064" layer="1"/>
-<wire x1="4.9784" y1="10.9982" x2="6.9342" y2="13.0048" width="0" layer="19" extent="1-1"/>
+<contactref element="R4" pad="1"/>
 </signal>
 <signal name="D-">
@@
 <contactref element="C1" pad="1"/>
 <contactref element="C2" pad="+"/>
-<wire x1="4.288" y1="4.859" x2="4.288" y2="5.9482" width="0.3048" layer="1"/>
-<wire x1="4.288" y1="5.9482" x2="4.2926" y2="5.9436" width="0.3048" layer="1"/>
-<wire x1="4.288" y1="5.9482" x2="3.8608" y2="6.3754" width="0.3048" layer="1"/>
-<wire x1="3.8608" y1="6.3754" x2="3.8608" y2="8.6868" width="0.3048" layer="1"/>
-<wire x1="3.8608" y1="8.6868" x2="2.286" y2="10.2616" width="0.3048" layer="1"/>
-<wire x1="2.286" y1="10.2616" x2="2.286" y2="12.102" width="0.3048" layer="1"/>
 <contactref element="U3" pad="1"/>
-<wire x1="1.8542" y1="22.5044" x2="1.8542" y2="14.4018" width="0.4064" layer="1"/>
-<wire x1="1.8542" y1="14.4018" x2="2.286" y2="13.97" width="0.4064" layer="1"/>
-<wire x1="2.286" y1="12.102" x2="2.286" y2="13.97" width="0.4064" layer="1"/>
+<wire x1="1.8542" y1="22.5044" x2="1.8542" y2="16.3576" width="0.4064" layer="1"/>
+<wire x1="1.8542" y1="16.3576" x2="2.286" y2="15.9258" width="0.4064" layer="1"/>
+<wire x1="2.286" y1="12.102" x2="2.286" y2="15.9258" width="0.4064" layer="1"/>
 <wire x1="1.8542" y1="22.5044" x2="1.8542" y2="25.8572" width="0.4064" layer="1"/>
 <wire x1="1.8542" y1="25.8572" x2="2.1844" y2="26.1874" width="0.4064" layer="1"/>
@@
 <wire x1="18.6816" y1="15.786" x2="18.2696" y2="15.374" width="0.4064" layer="1"/>
 <wire x1="17.3482" y1="15.374" x2="18.2696" y2="15.374" width="0.4064" layer="1"/>
+<wire x1="4.288" y1="4.859" x2="4.288" y2="8.2342" width="0.4064" layer="1"/>
+<wire x1="4.288" y1="8.2342" x2="2.286" y2="10.2362" width="0.4064" layer="1"/>
+<wire x1="2.286" y1="10.2362" x2="2.286" y2="12.102" width="0.4064" layer="1"/>
 </signal>
 <signal name="N$2">
@@
 <wire x1="9.4996" y1="11.049" x2="10.0186" y2="10.53" width="0.3048" layer="1"/>
 <wire x1="11.857" y1="10.53" x2="10.0186" y2="10.53" width="0.3048" layer="1"/>
-<wire x1="5.0292" y1="12.4968" x2="6.477" y2="11.049" width="0.3048" layer="1"/>
+<wire x1="5.1054" y1="12.4206" x2="6.477" y2="11.049" width="0.3048" layer="1"/>
 <wire x1="6.477" y1="11.049" x2="9.4996" y2="11.049" width="0.3048" layer="1"/>
-<wire x1="5.0292" y1="17.6276" x2="5.0292" y2="12.4968" width="0.3048" layer="1"/>
-<wire x1="5.0292" y1="17.6276" x2="6.9342" y2="19.5326" width="0.3048" layer="1"/>
+<wire x1="5.1054" y1="17.6784" x2="5.1054" y2="12.4206" width="0.3048" layer="1"/>
+<wire x1="5.1054" y1="17.6784" x2="6.9342" y2="19.5072" width="0.3048" layer="1"/>
 <contactref element="U3" pad="3"/>
-<wire x1="6.9342" y1="22.5044" x2="6.9342" y2="19.5326" width="0.3048" layer="1"/>
+<wire x1="6.9342" y1="22.5044" x2="6.9342" y2="19.5072" width="0.3048" layer="1"/>
 </signal>
 <signal name="SDA">
@@
 <wire x1="10.3084" y1="11.18" x2="9.8044" y2="11.684" width="0.3048" layer="1"/>
 <wire x1="9.8044" y1="11.684" x2="6.731" y2="11.684" width="0.3048" layer="1"/>
-<wire x1="6.731" y1="11.684" x2="5.6896" y2="12.7254" width="0.3048" layer="1"/>
-<wire x1="5.6896" y1="12.7254" x2="5.6896" y2="17.3482" width="0.3048" layer="1"/>
+<wire x1="6.731" y1="11.684" x2="5.7404" y2="12.6746" width="0.3048" layer="1"/>
+<wire x1="5.7404" y1="12.6746" x2="5.7404" y2="17.399" width="0.3048" layer="1"/>
 <contactref element="U3" pad="4"/>
-<wire x1="5.6896" y1="17.3482" x2="7.6708" y2="19.3294" width="0.3048" layer="1"/>
+<wire x1="5.7404" y1="17.399" x2="7.6708" y2="19.3294" width="0.3048" layer="1"/>
 <wire x1="7.6708" y1="19.3294" x2="9.0678" y2="19.3294" width="0.3048" layer="1"/>
 <wire x1="9.0678" y1="19.3294" x2="9.4742" y2="19.7358" width="0.3048" layer="1"/>
@@
 <wire x1="15.24" y1="11.4808" x2="15.24" y2="12.2174" width="0.3048" layer="1"/>
 </signal>
+<signal name="N$1">
+<contactref element="U3" pad="2"/>
+<contactref element="R4" pad="2"/>
+<wire x1="4.3942" y1="22.5044" x2="4.3942" y2="18.7452" width="0.6096" layer="1"/>
+<wire x1="4.3942" y1="18.7452" x2="3.99" y2="18.341" width="0.6096" layer="1"/>
+<wire x1="3.99" y1="14.6812" x2="3.99" y2="18.341" width="0.6096" layer="1"/>
+<polygon width="0.254" layer="1" isolate="0.4064">
+<vertex x="2.54" y="19.05"/>
+<vertex x="2.4638" y="7.3152"/>
+<vertex x="6.0706" y="7.2898"/>
+<vertex x="6.1214" y="19.05"/>
+<vertex x="5.3594" y="19.0246"/>
+<vertex x="2.5654" y="19.0246"/>
+</polygon>
+</signal>
 </signals>
