File: hardware/stm8-accelerometer -1.sch (EAGLE design)
At the start: 15 parts, among them U1 MCP1700T-3302E, U2 STM8SX03F3, U3 MPU6050

Commit message: Clean up.  Still WIP
Parts:
- added R4: 0R, ipc-7351-resistor:RESISTOR_1206
Connections:
- new net N$1: R4.2, U3.GND
- net GND: now also R4.1; no longer U3.GND
Changed lines of the file:
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@@
 <part name="U3" library="misc pcb" deviceset="MPU6050" device=""/>
 <part name="LICENSE1" library="Misc logo" deviceset="CC-BY" device="50%"/>
+<part name="R4" library="ipc-7351-resistor" deviceset="RESISTOR_" device="1206" value="0R"/>
 </parts>
 <sheets>
@@
 <instance part="SUPPLY7" gate="+3.3V" x="99.06" y="127"/>
 <instance part="H1" gate="G$1" x="213.36" y="93.98"/>
-<instance part="SUPPLY9" gate="GND" x="205.74" y="114.3"/>
+<instance part="SUPPLY9" gate="GND" x="205.74" y="106.68"/>
 <instance part="U3" gate="G$1" x="223.52" y="139.7"/>
 <instance part="LICENSE1" gate="G$1" x="132.08" y="5.08"/>
+<instance part="R4" gate="G$1" x="205.74" y="114.3" rot="R90"/>
 </instances>
 <busses>
@@
 <segment>
 <pinref part="SUPPLY9" gate="GND" pin="GND"/>
-<wire x1="210.82" y1="149.86" x2="205.74" y2="149.86" width="0.1524" layer="91"/>
-<wire x1="205.74" y1="149.86" x2="205.74" y2="116.84" width="0.1524" layer="91"/>
-<pinref part="U3" gate="G$1" pin="GND"/>
+<pinref part="R4" gate="G$1" pin="1"/>
 </segment>
 </net>
@@
 </segment>
 </net>
+<net name="N$1" class="0">
+<segment>
+<wire x1="210.82" y1="149.86" x2="205.74" y2="149.86" width="0.1524" layer="91"/>
+<wire x1="205.74" y1="149.86" x2="205.74" y2="119.38" width="0.1524" layer="91"/>
+<pinref part="U3" gate="G$1" pin="GND"/>
+<pinref part="R4" gate="G$1" pin="2"/>
+</segment>
+</net>
